File: boards/SmartInsolePCB/DesignESP32PCB.kicad_pcb (KiCad board)
At the start: 2 copper layers, 51 x 81.5 mm, 60 parts, among them J1 PJS008U-3000-0, J10 Conn_01x02_Pin, J11 Conn_01x02_Pin, J12 Conn_01x02_Pin, J13 Conn_01x05_Socket, J2 Conn_01x02_Pin, J3 Conn_01x02_Pin, J4 Conn_01x02_Pin, J5 Conn_01x02_Pin, J6 Conn_01x02_Pin, J7 Conn_01x02_Pin, J8 Conn_01x02_Pin, J9 Conn_01x02_Pin, Q1 SS8050-G, Q2 SS8050-G, SW1 B3F-4000, SW2 B3F-4000, SW3 B3F-4000, SW4 B3F-4000, U1 D3V3XA4B10LP, U2 ESP32-S3-WROOM-1, U3 MPU-6050, U4 TLV75801PDRV

Commit message: put extra comp on board
Parts:
- moved JP1 43.3 mm to (125.8, 71.1)
- moved R21 38.2 mm to (127.0, 61.0)
- moved R22 36.3 mm to (127.0, 66.0)
Routing:
- net /3V3: track 51.0 -> 100.0 mm
- net /GPIO0_STRAPPING: track 36.1 -> 68.4 mm
- net Net-(JP1-C): track 0.00 -> 5.24 mm
Changed lines of the file:
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@@
 		(tags "resistor")
 		(property "Reference" "R25"
-			(at 0 -1.43 270)
+			(at 0 -1.43 -90)
 			(layer "F.SilkS")
 			(effects
@@
 		)
 		(property "Value" "10k"
-			(at 0 1.43 270)
+			(at 0 1.43 -90)
 			(layer "F.Fab")
 			(effects
@@
 		)
 		(fp_text user "${REFERENCE}"
-			(at 0 0 270)
+			(at 0 0 -90)
 			(layer "F.Fab")
 			(effects
@@
 	(footprint "Jumper:SolderJumper-3_P2.0mm_Open_TrianglePad1.0x1.5mm"
 		(layer "F.Cu")
-		(at 161.7664 95.1992)
+		(at 125.8 71.12)
 		(descr "SMD Solder Jumper, 1x1.5mm Triangular Pads, 0.3mm gap, open")
 		(tags "solder jumper open")
@@
 		)
 		(property "Value" "10k"
-			(at 0 1.43 270)
+			(at 0 1.43 -90)
 			(layer "F.Fab")
 			(effects
@@
 		)
 		(fp_text user "${REFERENCE}"
-			(at 0 0 270)
+			(at 0 0 -90)
 			(layer "F.Fab")
 			(effects
@@
 		)
 		(property "Value" "10k"
-			(at 0 1.43 270)
+			(at 0 1.43 -90)
 			(layer "F.Fab")
 			(effects
@@
 		)
 		(fp_text user "${REFERENCE}"
-			(at 0 0 270)
+			(at 0 0 -90)
 			(layer "F.Fab")
 			(effects
@@
 	(footprint "Resistor_SMD:R_0603_1608Metric"
 		(layer "F.Cu")
-		(at 152.0364 89.7592)
+		(at 127 60.96)
 		(descr "Resistor SMD 0603 (1608 Metric), square (rectangular) end terminal, IPC_7351 nominal, (Body size source: IPC-SM-782 page 72, https://www.pcb-3d.com/wordpress/wp-content/uploads/ipc-sm-782a_amendment_1_and_2.pdf), generated with kicad-footprint-generator")
 		(tags "resistor")
@@
 	(footprint "Resistor_SMD:R_0603_1608Metric"
 		(layer "F.Cu")
-		(at 152.0364 92.2692)
+		(at 127 66.04)
 		(descr "Resistor SMD 0603 (1608 Metric), square (rectangular) end terminal, IPC_7351 nominal, (Body size source: IPC-SM-782 page 72, https://www.pcb-3d.com/wordpress/wp-content/uploads/ipc-sm-782a_amendment_1_and_2.pdf), generated with kicad-footprint-generator")
 		(tags "resistor")
@@
 		)
 		(property "Value" "10k"
-			(at 0 1.43 270)
+			(at 0 1.43 -90)
 			(layer "F.Fab")
 			(effects
@@
 		)
 		(fp_text user "${REFERENCE}"
-			(at 0 0 270)
+			(at 0 0 -90)
 			(layer "F.Fab")
 			(effects
@@
 	)
 	(segment
+		(start 127 66.402648)
+		(end 127 61.785)
+		(width 0.3)
+		(layer "F.Cu")
+		(net 3)
+	)
+	(segment
 		(start 129.7 105)
 		(end 127.9 105)
@@
 	)
 	(segment
+		(start 127.8 67.202648)
+		(end 127 66.402648)
+		(width 0.3)
+		(layer "F.Cu")
+		(net 3)
+	)
+	(segment
 		(start 126.3025 104.39)
 		(end 126.3845 104.472)
@@
 	)
 	(segment
+		(start 121.92 45.72)
+		(end 127.825 51.625)
+		(width 0.3)
+		(layer "F.Cu")
+		(net 3)
+	)
+	(segment
 		(start 126.2525 104.34)
 		(end 126.3025 104.39)
@@
 	)
 	(segment
+		(start 127 61.785)
+		(end 127.825 60.96)
+		(width 0.3)
+		(layer "F.Cu")
+		(net 3)
+	)
+	(segment
+		(start 106.68 46.536)
+		(end 107.496 45.72)
+		(width 0.3)
+		(layer "F.Cu")
+		(net 3)
+	)
+	(segment
 		(start 122.555 107.569)
 		(end 122.555 106.003)
@@
 	)
 	(segment
+		(start 127.825 51.625)
+		(end 127.825 60.96)
+		(width 0.3)
+		(layer "F.Cu")
+		(net 3)
+	)
+	(segment
+		(start 107.496 45.72)
+		(end 121.92 45.72)
+		(width 0.3)
+		(layer "F.Cu")
+		(net 3)
+	)
+	(segment
 		(start 114.7064 90.932)
 		(end 115.824 92.0496)
@@
 	)
 	(segment
+		(start 110.182 50.038)
+		(end 106.68 46.536)
+		(width 0.3)
+		(layer "F.Cu")
+		(net 3)
+	)
+	(segment
+		(start 127.8 71.12)
+		(end 127.8 67.202648)
+		(width 0.3)
+		(layer "F.Cu")
+		(net 3)
+	)
+	(segment
 		(start 127.9 105)
 		(end 127.29 104.39)
@@
 	)
 	(segment
+		(start 125.8 66.415)
+		(end 126.175 66.04)
+		(width 0.25)
+		(layer "F.Cu")
+		(net 88)
+	)
+	(segment
+		(start 125.8 71.12)
+		(end 125.8 66.415)
+		(width 0.25)
+		(layer "F.Cu")
+		(net 88)
+	)
+	(segment
 		(start 133.1926 111.252)
 		(end 132.1498 110.2092)
@@
 	)
 	(segment
+		(start 117.7148 94.9056)
+		(end 117.7148 78.14525)
+		(width 0.3)
+		(layer "B.Cu")
+		(net 98)
+	)
+	(segment
 		(start 129.2352 111.8108)
 		(end 121.0564 119.9896)
@@
 		(width 0.3)
 		(layer "B.Cu")
+		(net 98)
+	)
+	(segment
+		(start 117.7148 78.14525)
+		(end 124.74005 71.12)
+		(width 0.3)
+		(layer "B.Cu")
+		(net 98)
+	)
+	(segment
+		(start 121.6152 98.806)
+		(end 117.7148 94.9056)
+		(width 0.3)
+		(layer "B.Cu")

Commit message: down to 56
Routing:
- net /ESP32_EN: track 69.9 -> 71.2 mm
- net Net-(Q1-Pad3): track 12.5 -> 13.6 mm
- net Net-(C2-Pad1): track 28.3 -> 27.3 mm
- net GND: track 18.6 -> 19.3 mm

Commit message: 2 missing connections and 16 erros
Routing:
- net /RX: track 63.2 -> 33.2 mm
Changed lines of the file:
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@@
+	)
+	(segment
+		(start 141.75 116.4156)
+		(end 141.75 112.7)
+		(width 0.3)
+		(layer "B.Cu")
+		(net 48)
 	)
 	(segment
 		(start 119.634 78.4352)
 		(end 137.4502 78.4352)
-		(width 0.25)
-		(layer "B.Cu")
-		(net 48)
-	)
-	(segment
-		(start 141.645 116.5206)
-		(end 141.0716 117.094)
 		(width 0.25)
 		(layer "B.Cu")
@@
 	)
 	(segment
-		(start 141.645 82.63)
-		(end 141.645 116.5206)
-		(width 0.25)
+		(start 141.0716 117.094)
+		(end 141.75 116.4156)
+		(width 0.3)
 		(layer "B.Cu")
 		(net 48)

Commit message: saved work
Routing:
- net /GPIO46_STRAPPING: track 0.00 -> 51.4 mm, vias 0 -> 2
- net /GPIO3_STRAPPING: track 0.00 -> 48.5 mm, vias 0 -> 2
- net /3V3: track 100.0 -> 140.9 mm, vias 4 -> 6
- net /RX: track 33.2 -> 64.0 mm
- net /GPIO8: track 4.66 -> 19.8 mm, vias 0 -> 2
- net GND: track 19.3 -> 25.5 mm
- net /ESP32_EN: track 71.2 -> 67.3 mm
- net /MISO: track 31.4 -> 35.1 mm
- net /GPIO0_STRAPPING: track 68.4 -> 72.0 mm, vias 3 -> 6
- net /RTS: track 17.7 -> 20.7 mm
- net /TX: track 58.2 -> 60.2 mm
- net /GPIO12: track 24.4 -> 25.2 mm
Other:
- board size 51 x 81.5 mm -> 54.2 x 81.5 mm
